File: v2/midiprog.sch (EAGLE design)
At the start: 56 parts, among them IC1 PIC18F4550_40, IC2 TPIC6B596N, IC3 78L05Z, IC4 TPIC6B596N, Q1 8MHz, Q2 2N2222A, Q3 2N2222A, Q4 2N2222A

Commit message: Decent layout; not great.
Parts:
- removed R25: 220, rcl:R-US_0207/10
- added R23: 220, rcl:R-US_0207/10
Connections:
- net BFX2 renamed N$63
- net BFX4 renamed N$61
- net BFX7 renamed N$49
- net BPR2 renamed N$57
- net BPR4 renamed N$55
- net BPR7 renamed N$51
- removed net BFX1: BTN_FX_CN.1, U$2.A0
- removed net BFX3: BTN_FX_CN.5, U$2.A2
- removed net BFX5: BTN_FX_CN.9, U$2.A4
- removed net BFX6: BTN_FX_CN.11, U$2.A5
- removed net BFX8: BTN_FX_CN.15, U$2.A7
- removed net BPR1: BTN_PR_CN.1, U$1.A0
- removed net BPR3: BTN_PR_CN.5, U$1.A2
- removed net BPR5: BTN_PR_CN.9, U$1.A4
- removed net BPR6: BTN_PR_CN.11, U$1.A5
- removed net BPR8: BTN_PR_CN.15, U$1.A7
- removed net N$19 (its old number): LED_FX_CN.9, R19.2
- removed net N$20 (its old number): LED_FX_CN.7, R18.2
- removed net N$21 (its old number): LED_FX_CN.5, R17.2
- removed net N$22 (its old number): LED_FX_CN.3, R16.2
- removed net N$23 (its old number): LED_FX_CN.1, R15.2
- new net N$10: LED_FX_CN.11, R17.2
- new net N$13: LED_FX_CN.5, R20.2
- new net N$14: LED_FX_CN.3, R21.2
- new net N$15: LED_FX_CN.1, R22.2
- new net N$3: LED_FX_CN.13, R16.2
- new net N$46: BTN_FX_CN.9, U$2.A5
- new net N$47: BTN_PR_CN.9, U$1.A5
- new net N$48: BTN_FX_CN.11, U$2.A7
- new net N$50: BTN_PR_CN.11, U$1.A7
- new net N$52: BTN_PR_CN.15, U$1.A4
- new net N$56: BTN_PR_CN.5, U$1.A0
- new net N$58: BTN_PR_CN.1, U$1.A2
- new net N$60: BTN_FX_CN.15, U$2.A4
- new net N$62: BTN_FX_CN.5, U$2.A0
- new net N$64: BTN_FX_CN.1, U$2.A2
- net N$11: now also LED_FX_CN.9, R18.2; no longer LED_FX_CN.13, R21.2
- net N$12: now also LED_FX_CN.7, R19.2; no longer LED_FX_CN.11, R20.2
- net N$2: now also R15.2; no longer R22.2
- net N$24: now also R3.2; no longer R12.2
- net N$27: now also R4.2; no longer R7.2
- net N$30: now also R7.2; no longer R4.2
- net N$32: now also R12.2; no longer R3.2
- net N$36: now also R13.2; no longer R2.2
- net N$37: now also R23.2; no longer R25.2
- net N$38: now also IC2G$1.Q0, R2.1; no longer IC2G$1.Q7, R13.1
- net N$39: now also IC2G$1.Q1, R3.1; no longer IC2G$1.Q6, R12.1
- net N$40: now also IC2G$1.Q2, R4.1; no longer IC2G$1.Q5, R7.1
- net N$41: now also IC2G$1.Q3; no longer IC2G$1.Q4
- net N$42: now also IC2G$1.Q4, R7.1; no longer IC2G$1.Q3, R4.1
- net N$43: now also IC2G$1.Q5, R12.1; no longer IC2G$1.Q2, R3.1
- net N$44: now also IC2G$1.Q6, R13.1; no longer IC2G$1.Q1, R2.1
- net N$45: now also IC2G$1.Q7, R23.1; no longer IC2G$1.Q0, R25.1
- net N$6: now also R2.2; no longer R13.2
Other:
- moved on the sheet: BTN_FX_CN, BTN_PR_CN, C8, C9, IC2, IC2P, IC4, IC4P, LED_FX_CN, LED_PR_CN, Q4, R12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

Commit message: Added custom package for 7805.
Parts:
- removed 9V_BATT: (no value), con-amp-quick:M02
- removed C6, C7: 10u, rcl:C-US050-025X075
- removed D1: 1N4001, diode:1N4004
- removed IC3: 78L05Z, linear:78L05Z
- removed Q1: 8MHz, special:XTAL
- added C10, C11: 10u, rcl:CPOL-USE2.5-6
- added Q5: 8MHz, special:XTAL/S
- added U$3: 7805, 7805:7805
Connections:
- removed net N$33: 9V_BATT.2, D1.A
- net +9V: now also C10.+, U$3.VI; no longer C6.1, IC3.VI
- net GND: now also C10.-, C11.-, U$3.GND; no longer 9V_BATT.1, C6.2, C7.2, IC3.GND
- net N$35: no longer D1.C
- net OSC1: now also Q5.2; no longer Q1.2
- net OSC2: now also Q5.1; no longer Q1.1
- net VDD: now also C11.+, U$3.VO; no longer C7.1, IC3.VO

Commit message: Added correct parts from SparkFun to schematic and board.
Parts:
- removed MIDI_CN: (no value), con-amp-quick:MA05
- removed X1: (no value), con-berg:PN61729
- added JP1: USB-B, SparkFun-Connectors-fdb4deb3ddf02d02cecaec8c0f5c972a585683b1:USBPTH
- added MIDI_OUT: MIDI_CONN_FEMALE_SUPPORT, SparkFun-Connectors-fdb4deb3ddf02d02cecaec8c0f5c972a585683b1:MIDI_CONN_FEMALE_SUPPORT
Connections:
- net GND: now also JP1.GND, MIDI_OUT.NC2; no longer MIDI_CN.2, X1.4
- net N$8: now also MIDI_OUT.MIDI_IN; no longer MIDI_CN.5
- net N$9: now also MIDI_OUT.MIDI_OUT; no longer MIDI_CN.4
- net USB_D+: now also JP1.D+; no longer X1.3
- net USB_D-: now also JP1.D-; no longer X1.2
- net USB_VCC: now also JP1.VBUS; no longer X1.1
Other:
- moved on the sheet: TP1

Commit message: Added C6 and C7 to VDD off muxes.
Parts:
- added C6, C7: .1, rcl:C-US050-025X075
Connections:
- net GND: now also C6.2, C7.2
- net VDD: now also C6.1, C7.1
Changed lines of the file:
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@@
 <part name="MIDI_OUT" library="SparkFun-Connectors-fdb4deb3ddf02d02cecaec8c0f5c972a585683b1" deviceset="MIDI_CONN_FEMALE_SUPPORT" device=""/>
 <part name="JP1" library="SparkFun-Connectors-fdb4deb3ddf02d02cecaec8c0f5c972a585683b1" deviceset="USB" device="PTH" value="USB-B"/>
+<part name="C6" library="rcl" deviceset="C-US" device="050-025X075" value=".1"/>
+<part name="GND3" library="supply1" deviceset="GND" device=""/>
+<part name="C7" library="rcl" deviceset="C-US" device="050-025X075" value=".1"/>
+<part name="GND12" library="supply1" deviceset="GND" device=""/>
 </parts>
 <sheets>
@@
 <instance part="GND8" gate="1" x="401.32" y="27.94"/>
 <instance part="R11" gate="G$1" x="393.7" y="50.8"/>
-<instance part="VDD6" gate="G$1" x="381" y="152.4"/>
+<instance part="VDD6" gate="G$1" x="391.16" y="160.02"/>
 <instance part="GND9" gate="1" x="358.14" y="119.38"/>
 <instance part="VDD1" gate="G$1" x="248.92" y="63.5"/>
@@
 <instance part="C8" gate="G$1" x="195.58" y="119.38"/>
 <instance part="VDD12" gate="G$1" x="137.16" y="96.52" rot="R90"/>
-<instance part="VDD13" gate="G$1" x="294.64" y="152.4"/>
+<instance part="VDD13" gate="G$1" x="304.8" y="160.02"/>
 <instance part="GND16" gate="1" x="271.78" y="73.66"/>
 <instance part="U$2" gate="G$1" x="287.02" y="134.62"/>
@@
 <instance part="MIDI_OUT" gate="G$1" x="416.56" y="50.8" rot="R180"/>
 <instance part="JP1" gate="G$1" x="393.7" y="-2.54"/>
+<instance part="C6" gate="G$1" x="312.42" y="147.32"/>
+<instance part="GND3" gate="1" x="312.42" y="139.7"/>
+<instance part="C7" gate="G$1" x="398.78" y="147.32"/>
+<instance part="GND12" gate="1" x="398.78" y="139.7"/>
 </instances>
 <busses>
@@
 </segment>
 <segment>
-<wire x1="381" y1="142.24" x2="381" y2="149.86" width="0.1524" layer="91"/>
+<wire x1="381" y1="142.24" x2="391.16" y2="142.24" width="0.1524" layer="91"/>
+<wire x1="391.16" y1="142.24" x2="391.16" y2="152.4" width="0.1524" layer="91"/>
 <pinref part="VDD6" gate="G$1" pin="VDD"/>
 <pinref part="U$1" gate="G$1" pin="VCC"/>
+<wire x1="391.16" y1="152.4" x2="391.16" y2="157.48" width="0.1524" layer="91"/>
+<wire x1="391.16" y1="152.4" x2="398.78" y2="152.4" width="0.1524" layer="91"/>
+<wire x1="398.78" y1="152.4" x2="398.78" y2="149.86" width="0.1524" layer="91"/>
+<pinref part="C7" gate="G$1" pin="1"/>
+<junction x="391.16" y="152.4"/>
 </segment>
 <segment>
@@
 </segment>
 <segment>
-<wire x1="294.64" y1="142.24" x2="294.64" y2="149.86" width="0.1524" layer="91"/>
+<wire x1="294.64" y1="142.24" x2="304.8" y2="142.24" width="0.1524" layer="91"/>
+<wire x1="304.8" y1="142.24" x2="304.8" y2="152.4" width="0.1524" layer="91"/>
 <pinref part="VDD13" gate="G$1" pin="VDD"/>
 <pinref part="U$2" gate="G$1" pin="VCC"/>
+<wire x1="304.8" y1="152.4" x2="304.8" y2="157.48" width="0.1524" layer="91"/>
+<wire x1="304.8" y1="152.4" x2="312.42" y2="152.4" width="0.1524" layer="91"/>
+<wire x1="312.42" y1="152.4" x2="312.42" y2="149.86" width="0.1524" layer="91"/>
+<pinref part="C6" gate="G$1" pin="1"/>
+<junction x="304.8" y="152.4"/>
 </segment>
 <segment>
@@
 <junction x="274.32" y="76.2"/>
 </segment>
+<segment>
+<pinref part="C6" gate="G$1" pin="2"/>
+<pinref part="GND3" gate="1" pin="GND"/>
+</segment>
+<segment>
+<pinref part="C7" gate="G$1" pin="2"/>
+<pinref part="GND12" gate="1" pin="GND"/>
+</segment>
 </net>

Commit message: More clearance between button headers and mux chips. Moved timing crystal closer to PIC. Swapped C11 and C2 positions. Swapped MIDI OUT pins.
Connections:
- net N$8: now also R11.2; no longer R10.2
- net N$9: now also R10.2; no longer R11.2
Changed lines of the file:
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@@
-</segment>
-</net>
-<net name="N$8" class="0">
-<segment>
-<wire x1="403.86" y1="45.72" x2="396.24" y2="45.72" width="0.1524" layer="91"/>
-<pinref part="R10" gate="G$1" pin="2"/>
-<pinref part="MIDI_OUT" gate="G$1" pin="MIDI_IN"/>
 </segment>
 </net>
@@
 </segment>
 </net>
-<net name="N$9" class="0">
-<segment>
-<wire x1="403.86" y1="48.26" x2="398.78" y2="48.26" width="0.1524" layer="91"/>
-<wire x1="398.78" y1="48.26" x2="398.78" y2="50.8" width="0.1524" layer="91"/>
-<pinref part="R11" gate="G$1" pin="2"/>
-<pinref part="MIDI_OUT" gate="G$1" pin="MIDI_OUT"/>
-</segment>
-</net>
 <net name="N$34" class="0">
 <segment>
@@
 </segment>
 </net>
+<net name="N$8" class="0">
+<segment>
+<pinref part="R11" gate="G$1" pin="2"/>
+<wire x1="398.78" y1="50.8" x2="398.78" y2="45.72" width="0.1524" layer="91"/>
+<pinref part="MIDI_OUT" gate="G$1" pin="MIDI_IN"/>
+<wire x1="398.78" y1="45.72" x2="403.86" y2="45.72" width="0.1524" layer="91"/>
+</segment>
+</net>
+<net name="N$9" class="0">
+<segment>
+<pinref part="R10" gate="G$1" pin="2"/>
+<wire x1="396.24" y1="45.72" x2="396.24" y2="48.26" width="0.1524" layer="91"/>
+<pinref part="MIDI_OUT" gate="G$1" pin="MIDI_OUT"/>
+<wire x1="396.24" y1="48.26" x2="403.86" y2="48.26" width="0.1524" layer="91"/>
+</segment>
+</net>

Commit message: Fixed the MIDI part
Connections:
- net GND: now also MIDI_OUT.GND; no longer MIDI_OUT.NC2
- net N$8: now also MIDI_OUT.CSRC; no longer MIDI_OUT.MIDI_IN
- net N$9: now also MIDI_OUT.CSNK; no longer MIDI_OUT.MIDI_OUT
- net SHIFTREG_D: now also IC1.RA3/AN3/VREF+; no longer IC1.RA3/AN4/VREF+
Changed lines of the file:
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@@
 <wire x1="401.32" y1="53.34" x2="403.86" y2="53.34" width="0.1524" layer="91"/>
 <pinref part="GND8" gate="1" pin="GND"/>
-<pinref part="MIDI_OUT" gate="G$1" pin="NC2"/>
+<pinref part="MIDI_OUT" gate="G$1" pin="GND"/>
 </segment>
 <segment>
@@
 <segment>
 <wire x1="251.46" y1="33.02" x2="241.3" y2="33.02" width="0.1524" layer="91"/>
-<pinref part="IC1" gate="G$1" pin="RA3/AN4/VREF+"/>
+<pinref part="IC1" gate="G$1" pin="RA3/AN3/VREF+"/>
 <label x="241.3" y="33.02" size="1.778" layer="95" rot="R180" xref="yes"/>
 </segment>
@@
 <pinref part="R11" gate="G$1" pin="2"/>
 <wire x1="398.78" y1="50.8" x2="398.78" y2="45.72" width="0.1524" layer="91"/>
-<pinref part="MIDI_OUT" gate="G$1" pin="MIDI_IN"/>
+<pinref part="MIDI_OUT" gate="G$1" pin="CSRC"/>
 <wire x1="398.78" y1="45.72" x2="403.86" y2="45.72" width="0.1524" layer="91"/>
 </segment>
@@
 <pinref part="R10" gate="G$1" pin="2"/>
 <wire x1="396.24" y1="45.72" x2="396.24" y2="48.26" width="0.1524" layer="91"/>
-<pinref part="MIDI_OUT" gate="G$1" pin="MIDI_OUT"/>
+<pinref part="MIDI_OUT" gate="G$1" pin="CSNK"/>
 <wire x1="396.24" y1="48.26" x2="403.86" y2="48.26" width="0.1524" layer="91"/>
 </segment>

Commit message: Renamed library file.
Parts:
- JP1: device SparkFun-Connectors-fdb4deb3ddf02d02cecaec8c0f5c972a585683b1:USBPTH -> SparkFun-Connectors:USBPTH
- MIDI_OUT: device SparkFun-Connectors-fdb4deb3ddf02d02cecaec8c0f5c972a585683b1:MIDI_CONN_FEMALE_SUPPORT -> SparkFun-Connectors:MIDI_CONN_FEMALE_SUPPORT
Changed lines of the file:
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@@
 <part name="C11" library="rcl" deviceset="CPOL-US" device="E2.5-6" value="10u"/>
 <part name="U$3" library="7805" deviceset="7805" device=""/>
-<part name="MIDI_OUT" library="SparkFun-Connectors-fdb4deb3ddf02d02cecaec8c0f5c972a585683b1" deviceset="MIDI_CONN_FEMALE_SUPPORT" device=""/>
-<part name="JP1" library="SparkFun-Connectors-fdb4deb3ddf02d02cecaec8c0f5c972a585683b1" deviceset="USB" device="PTH" value="USB-B"/>
+<part name="MIDI_OUT" library="SparkFun-Connectors" deviceset="MIDI_CONN_FEMALE_SUPPORT" device=""/>
+<part name="JP1" library="SparkFun-Connectors" deviceset="USB" device="PTH" value="USB-B"/>
 <part name="C6" library="rcl" deviceset="C-US" device="050-025X075" value=".1"/>
 <part name="GND3" library="supply1" deviceset="GND" device=""/>
